File: kicad/PaperBot_RGB/PaperBot.kicad_pcb (KiCad board)
At the start: 2 copper layers, 60.7 x 49.4 mm, 7 parts, among them U2 BAT_HLD_SMD

Commit message: V 19.11.2024
Parts:
- added S2: Micro_Schalter, !Goody:Micro_SchalterKHF, F.Cu at (100.9, 80.1)
- moved M- 12.8 mm to (138.3, 67.4)
- renumbered M- to M+, M+ to M-
Connections:
- M+ pad 1: Net-(D1-K) -> Net-(D1-A)
- M- pad 1: Net-(D1-A) -> Net-(D1-K)
- U2 pad 1: (no net) -> Net-(S1-A-Pad1)
Routing:
- net Net-(S1-A-Pad1): track 19.8 -> 34.0 mm
- net Net-(D1-A): track 65.1 -> 73.4 mm
- net Net-(D1-K): track 66.1 -> 64.6 mm
Other:
- board text added: "KHF 11.2024"
- board text added: "LED"
- board text added: "M"
- board text added: "PaperBot"
- board text removed: "KHF 07.2024"
Changed lines of the file:
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@@
       (drillshape 0)
       (scaleselection 1)
-      (outputdirectory "../PaperBotGerber/")
+      (outputdirectory "PaperBotGerber/")
     )
   )
@@
   (net 4 "unconnected-(S1-A-Pad3)")
   (footprint "!Goody:LP_rund" (layer "F.Cu")
-    (at 151.1 67.25)
+    (at 138.3 67.4)
     (descr "LP")
     (attr through_hole)
-    (fp_text reference "M+" (at 0.1 2.1) (layer "B.SilkS")
-        (effects (font (size 1 1) (thickness 0.15)))
+    (fp_text reference "M-" (at 0.1 2.1) (layer "B.SilkS")
+        (effects (font (size 1 1) (thickness 0.15)) (justify mirror))
     )
     (fp_text value "LP_rund" (at 2.54 -6) (layer "F.Fab")
@@
     )
     (pad "1" thru_hole circle (at 0 0) (size 2 2) (drill 1.1) (layers "*.Cu" "*.Mask")
-      (net 2 "Net-(D1-A)"))
+      (net 1 "Net-(D1-K)"))
+  )
+  (footprint "!Goody:Micro_SchalterKHF" (layer "F.Cu")
+    (at 100.9 80.1 90)
+    (descr "Micro_SchalterKHF")
+    (property "Sheetfile" "PaperBot.kicad_sch")
+    (property "Sheetname" "")
+    (property "ki_description" "Micro_Schalter")
+    (attr through_hole)
+    (fp_text reference "S2" (at 1.4 3.5 90) (layer "User.1")
+        (effects (font (size 1 1) (thickness 0.15)))
+    )
+    (fp_text value "Micro_Schalter" (at 2.4 6 90) (layer "F.Fab")
+        (effects (font (size 1 1) (thickness 0.15)))
+    )
+    (fp_line (start -2.3876 -2.0066) (end 7.5692 -2.0066)
+      (stroke (width 0.12) (type solid)) (layer "F.SilkS"))
+    (fp_line (start -2.3876 1.9304) (end -2.413 -2.0066)
+      (stroke (width 0.12) (type solid)) (layer "F.SilkS"))
+    (fp_line (start 7.5692 -2.0066) (end 7.5692 1.9304)
+      (stroke (width 0.12) (type solid)) (layer "F.SilkS"))
+    (fp_line (start 7.5692 1.9304) (end -2.3876 1.9304)
+      (stroke (width 0.12) (type solid)) (layer "F.SilkS"))
+    (pad "1" thru_hole circle (at 0 0 90) (size 2 2) (drill 1) (layers "*.Cu" "*.Mask")
+      (net 3 "Net-(S1-A-Pad1)") (pinfunction "A") (pintype "passive"))
+    (pad "2" thru_hole circle (at 2.54 0 90) (size 2 2) (drill 1) (layers "*.Cu" "*.Mask")
+      (net 2 "Net-(D1-A)") (pinfunction "E") (pintype "passive"))
+    (pad "3" thru_hole circle (at 5.08 0 90) (size 2 2) (drill 1) (layers "*.Cu" "*.Mask")
+      (pinfunction "A") (pintype "passive+no_connect"))
   )
   (footprint "!Goody:ob-logo_B.SilkS" (layer "F.Cu")
@@
     (descr "LP")
     (attr through_hole)
-    (fp_text reference "M-" (at 0.25 2.65) (layer "B.SilkS")
-        (effects (font (size 1 1) (thickness 0.15)))
+    (fp_text reference "M+" (at 0.25 2.65) (layer "B.SilkS")
+        (effects (font (size 1 1) (thickness 0.15)) (justify mirror))
     )
     (fp_text value "LP_rund" (at 2.54 -6) (layer "F.Fab")
@@
     )
     (pad "1" thru_hole circle (at 0 0) (size 2 2) (drill 1.2) (layers "*.Cu" "*.Mask")
-      (net 1 "Net-(D1-K)"))
+      (net 2 "Net-(D1-A)"))
   )
   (footprint "LED_THT:LED_D5.0mm" (layer "F.Cu")
@@
       (net 3 "Net-(S1-A-Pad1)"))
     (pad "1" smd rect (at 12.94 -2.032 180) (size 5 2) (layers "B.Cu" "B.Paste" "B.Mask")
-      (pintype "power_out"))
+      (net 3 "Net-(S1-A-Pad1)") (pintype "power_out"))
     (pad "1" smd rect (at 12.94 1.524 180) (size 5 2) (layers "B.Cu" "B.Paste" "B.Mask")
-      (pintype "power_out"))
+      (net 3 "Net-(S1-A-Pad1)") (pintype "power_out"))
     (pad "2" smd circle (at 0 0 180) (size 17.78 17.78) (layers "B.Cu" "B.Paste" "B.Mask")
       (net 1 "Net-(D1-K)") (pintype "power_out"))
@@
   (gr_rect (start 154.4 73) (end 157.3 81.9)
     (stroke (width 0.15) (type default)) (fill none) (layer "B.SilkS"))
+  (gr_rect (start 99.4 72.9) (end 102.3 81.8)
+    (stroke (width 0.15) (type default)) (fill none) (layer "B.SilkS"))
   (gr_arc (start 99.989214 93.39) (mid 98.575 92.804214) (end 97.989214 91.39)
     (stroke (width 0.1) (type default)) (layer "Edge.Cuts"))
@@
   (gr_arc (start 156.64033 44.009937) (mid 158.054544 44.595723) (end 158.64033 46.009937)
     (stroke (width 0.1) (type default)) (layer "Edge.Cuts"))
-  (gr_text "KHF 07.2024" (at 133.9 57.55) (layer "B.Cu")
+  (gr_text "KHF 11.2024" (at 133.9 57.55) (layer "B.Cu")
     (effects (font (size 1 1) (thickness 0.15)) (justify left bottom mirror))
+  )
+  (gr_text "M" (at 100.9 71.1) (layer "B.SilkS")
+    (effects (font (size 1 1) (thickness 0.15)))
   )
   (gr_text "K" (at 141.2 60.6) (layer "B.SilkS")
     (effects (font (size 1 1) (thickness 0.15)) (justify left bottom mirror))
   )
+  (gr_text "LED" (at 155.9 70.7) (layer "B.SilkS")
+    (effects (font (size 1 1) (thickness 0.15)) (justify mirror))
+  )
   (gr_text "JLCJLCJLCJLC" (at 153.38 91.73) (layer "B.SilkS")
     (effects (font (size 1 1) (thickness 0.15)) (justify left bottom mirror))
@@
     (effects (font (size 1 1) (thickness 0.15)) (justify left bottom mirror))
   )
+  (gr_text "PaperBot" (at 133.4 67.3) (layer "B.SilkS")
+    (effects (font (size 2 2) (thickness 0.3)) (justify left bottom mirror))
+  )
   (gr_text "K" (at 109.9 60.5) (layer "B.SilkS")
     (effects (font (size 1 1) (thickness 0.15)) (justify left bottom mirror))
   )
-  (gr_text "KHF 07.2024" (at 133.9 57.55) (layer "B.Mask")
+  (gr_text "KHF 11.2024" (at 133.9 57.55) (layer "B.Mask")
     (effects (font (size 1 1) (thickness 0.15)) (justify left bottom mirror))
   )
+  (segment (start 142.62 67.4) (end 142.96 67.74) (width 0.25) (layer "B.Cu") (net 1))
   (segment (start 142.96 60) (end 142.96 67.74) (width 0.25) (layer "B.Cu") (net 1))
-  (segment (start 111.6 67.5) (end 105.3 67.5) (width 0.25) (layer "B.Cu") (net 1))
+  (segment (start 138.3 67.4) (end 142.62 67.4) (width 0.25) (layer "B.Cu") (net 1))
   (segment (start 142.96 67.74) (end 127.4 83.3) (width 0.25) (layer "B.Cu") (net 1))
   (segment (start 111.6 59.8) (end 111.6 67.5) (width 0.25) (layer "B.Cu") (net 1))
   (segment (start 111.6 67.5) (end 127.4 83.3) (width 0.25) (layer "B.Cu") (net 1))
+  (segment (start 105.3 76.6) (end 104.34 77.56) (width 0.25) (layer "B.Cu") (net 2))
   (segment (start 116.65 59.8) (end 121.5 54.95) (width 0.25) (layer "B.Cu") (net 2))
-  (segment (start 145.51 67.25) (end 151.1 67.25) (width 0.25) (layer "B.Cu") (net 2))
   (segment (start 114.14 59.8) (end 116.65 59.8) (width 0.25) (layer "B.Cu") (net 2))
   (segment (start 145.5 67.26) (end 145.5 60) (width 0.25) (layer "B.Cu") (net 2))
@@
   (segment (start 155.9 77.66) (end 145.5 67.26) (width 0.25) (layer "B.Cu") (net 2))
   (segment (start 143.95 54.95) (end 145.5 56.5) (width 0.25) (layer "B.Cu") (net 2))
+  (segment (start 104.34 77.56) (end 100.9 77.56) (width 0.25) (layer "B.Cu") (net 2))
+  (segment (start 105.3 67.5) (end 105.3 76.6) (width 0.25) (layer "B.Cu") (net 2))
   (segment (start 121.5 54.95) (end 143.95 54.95) (width 0.25) (layer "B.Cu") (net 2))
   (segment (start 145.5 56.5) (end 145.5 60) (width 0.25) (layer "B.Cu") (net 2))
   (segment (start 154.324 81.776) (end 155.9 80.2) (width 0.25) (layer "B.Cu") (net 3))
   (segment (start 140.354 85.332) (end 140.354 81.776) (width 0.25) (layer "B.Cu") (net 3))
+  (segment (start 112.784 80.1) (end 114.46 81.776) (width 0.25) (layer "B.Cu") (net 3))
   (segment (start 140.354 81.776) (end 154.324 81.776) (width 0.25) (layer "B.Cu") (net 3))
+  (segment (start 100.9 80.1) (end 112.784 80.1) (width 0.25) (layer "B.Cu") (net 3))
 )

Commit message: V20112024
Parts:
- moved D1 0.25 mm to (111.3, 59.8)
- moved D2 0.25 mm to (142.7, 60.0)
Routing:
- net Net-(S1-A-Pad1): track 34.0 -> 37.6 mm
- net Net-(D1-K): track 64.6 -> 62.2 mm
Changed lines of the file:
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@@
         (effects (font (size 1 1) (thickness 0.15)) (justify mirror))
     )
-    (fp_text value "LP_rund" (at 2.54 -6) (layer "F.Fab")
+    (fp_text value "LP_rund" (at 2.29 -6.01) (layer "F.Fab")
         (effects (font (size 1 1) (thickness 0.15)))
     )
@@
   )
   (footprint "LED_THT:LED_D5.0mm" (layer "F.Cu")
-    (at 142.96 60)
+    (at 142.71 59.99)
     (descr "LED, diameter 5.0mm, 2 pins, http://cdn-reichelt.de/documents/datenblatt/A500/LL-504BC2E-009.pdf")
     (tags "LED diameter 5.0mm 2 pins")
@@
         (effects (font (size 1 1) (thickness 0.15)) (justify mirror))
     )
-    (fp_text value "LP_rund" (at 2.54 -6) (layer "F.Fab")
+    (fp_text value "LP_rund" (at 2.29 -6.01) (layer "F.Fab")
         (effects (font (size 1 1) (thickness 0.15)))
     )
@@
   )
   (footprint "LED_THT:LED_D5.0mm" (layer "F.Cu")
-    (at 111.6 59.8)
+    (at 111.35 59.79)
     (descr "LED, diameter 5.0mm, 2 pins, http://cdn-reichelt.de/documents/datenblatt/A500/LL-504BC2E-009.pdf")
     (tags "LED diameter 5.0mm 2 pins")
@@
     (effects (font (size 1 1) (thickness 0.15)))
   )
-  (gr_text "K" (at 141.2 60.6) (layer "B.SilkS")
+  (gr_text "K" (at 140.95 60.59) (layer "B.SilkS")
     (effects (font (size 1 1) (thickness 0.15)) (justify left bottom mirror))
   )
@@
     (effects (font (size 2 2) (thickness 0.3)) (justify left bottom mirror))
   )
-  (gr_text "K" (at 109.9 60.5) (layer "B.SilkS")
+  (gr_text "K" (at 109.65 60.49) (layer "B.SilkS")
     (effects (font (size 1 1) (thickness 0.15)) (justify left bottom mirror))
   )
@@
     (effects (font (size 1 1) (thickness 0.15)) (justify left bottom mirror))
   )
-  (segment (start 142.62 67.4) (end 142.96 67.74) (width 0.25) (layer "B.Cu") (net 1))
-  (segment (start 142.96 60) (end 142.96 67.74) (width 0.25) (layer "B.Cu") (net 1))
-  (segment (start 138.3 67.4) (end 142.62 67.4) (width 0.25) (layer "B.Cu") (net 1))
-  (segment (start 142.96 67.74) (end 127.4 83.3) (width 0.25) (layer "B.Cu") (net 1))
-  (segment (start 111.6 59.8) (end 111.6 67.5) (width 0.25) (layer "B.Cu") (net 1))
-  (segment (start 111.6 67.5) (end 127.4 83.3) (width 0.25) (layer "B.Cu") (net 1))
+  (segment (start 142.71 66.82) (end 142.13 67.4) (width 0.25) (layer "B.Cu") (net 1))
+  (segment (start 111.35 67.49) (end 111.59 67.49) (width 0.25) (layer "B.Cu") (net 1))
+  (segment (start 138.3 72.4) (end 127.4 83.3) (width 0.25) (layer "B.Cu") (net 1))
+  (segment (start 138.3 67.4) (end 138.3 72.4) (width 0.25) (layer "B.Cu") (net 1))
+  (segment (start 142.71 59.99) (end 142.71 66.82) (width 0.25) (layer "B.Cu") (net 1))
+  (segment (start 111.59 67.49) (end 127.4 83.3) (width 0.25) (layer "B.Cu") (net 1))
+  (segment (start 142.13 67.4) (end 138.3 67.4) (width 0.25) (layer "B.Cu") (net 1))
+  (segment (start 111.35 59.79) (end 111.35 67.49) (width 0.25) (layer "B.Cu") (net 1))
+  (segment (start 145.49 67.25) (end 145.25 67.25) (width 0.25) (layer "B.Cu") (net 2))
   (segment (start 105.3 76.6) (end 104.34 77.56) (width 0.25) (layer "B.Cu") (net 2))
-  (segment (start 116.65 59.8) (end 121.5 54.95) (width 0.25) (layer "B.Cu") (net 2))
-  (segment (start 114.14 59.8) (end 116.65 59.8) (width 0.25) (layer "B.Cu") (net 2))
-  (segment (start 145.5 67.26) (end 145.5 60) (width 0.25) (layer "B.Cu") (net 2))
-  (segment (start 145.5 67.26) (end 145.51 67.25) (width 0.25) (layer "B.Cu") (net 2))
-  (segment (start 155.9 77.66) (end 145.5 67.26) (width 0.25) (layer "B.Cu") (net 2))
-  (segment (start 143.95 54.95) (end 145.5 56.5) (width 0.25) (layer "B.Cu") (net 2))
+  (segment (start 116.4 59.79) (end 113.89 59.79) (width 0.25) (layer "B.Cu") (net 2))
+  (segment (start 121.25 54.94) (end 116.4 59.79) (width 0.25) (layer "B.Cu") (net 2))
+  (segment (start 145.25 67.25) (end 145.25 59.99) (width 0.25) (layer "B.Cu") (net 2))
+  (segment (start 145.25 56.25) (end 143.94 54.94) (width 0.25) (layer "B.Cu") (net 2))
+  (segment (start 145.25 59.99) (end 145.25 56.25) (width 0.25) (layer "B.Cu") (net 2))
   (segment (start 104.34 77.56) (end 100.9 77.56) (width 0.25) (layer "B.Cu") (net 2))
   (segment (start 105.3 67.5) (end 105.3 76.6) (width 0.25) (layer "B.Cu") (net 2))
-  (segment (start 121.5 54.95) (end 143.95 54.95) (width 0.25) (layer "B.Cu") (net 2))
-  (segment (start 145.5 56.5) (end 145.5 60) (width 0.25) (layer "B.Cu") (net 2))
+  (segment (start 155.9 77.66) (end 145.49 67.25) (width 0.25) (layer "B.Cu") (net 2))
+  (segment (start 143.94 54.94) (end 121.25 54.94) (width 0.25) (layer "B.Cu") (net 2))
+  (segment (start 114.46 85.332) (end 114.46 81.776) (width 0.25) (layer "B.Cu") (net 3))
   (segment (start 154.324 81.776) (end 155.9 80.2) (width 0.25) (layer "B.Cu") (net 3))
   (segment (start 140.354 85.332) (end 140.354 81.776) (width 0.25) (layer "B.Cu") (net 3))
